Commit message: docs(essential): complete deep lecture notes, lab sheets, and rubrics for all 16 weeks

File: Essential_ROS/Week_08_Midterm_Practical_Exam/solution/solution_urdf.urdf (robot description, URDF)
Before this commit: robot diff_drive_robot, 9 links, 8 joints
Links:
- link base_link: mass 5.0 -> 8.0; geometry collision box size=0.50 0.30 0.15; visual box size=0.50 0.30 0.15
- link left_wheel_link: mass 0.75 -> 0.80
- link right_wheel_link: mass 0.75 -> 0.80
