Commit message: feat: make every lab a tested ROS 2 package with real run results
Turn all 16 Essential weeks and 6 Advanced modules into ament_python
packages (amr_week01..16, amr_adv01..06) built and tested in the
ros:lab-runner image (ROS 2 Jazzy, Gazebo Sim 8 Harmonic, headless).

- Replace fabricated terminal screenshots and transcripts with real
  run output (results/*.txt, real SLAM maps, paths, TF trees)
- Fix lab bugs found by running them: W07 wheel contact (odom yaw now
  matches ground truth), Nav2/SLAM/patrol/mission configs, ros2_control
  TwistStamped, opennav_docking actions, RMF fleet config, SROS2 enforce
- Advanced 06 capstone: one-command headless warehouse system with Nav2,
  collision_monitor StopZone, docking + AprilTag, KPI measurement vs
  Gazebo ground truth (5/5 runs pass), kidnapped-robot demo
- Start headless gz sim directly instead of via gz_sim.launch.py, whose
  sh wrapper left the gz server running after launch shutdown
- 260 automated tests (unit + launch_testing); Makefile (image, build,
  test, lint); CI builds the image and runs make lint/test
- Old Essential module folders become redirect stubs to the weeks;
  syllabi, weekly docs and READMEs aligned with the packages; relative
  links checked by scripts/check_links.py
- Docker: pinned base image, dist-upgrade, run as host uid, forward
  isolation env vars, core dumps disabled

Co-Authored-By: Claude Opus 5.5 <noreply@anthropic.com>

File: Advanced_ROS/01_ros2_control_Hardware/urdf/diff_drive_ros2_control.xacro (robot description, xacro)
@@ -1,38 +1,158 @@
 <?xml version="1.0"?>
-<robot xmlns:xacro="http://www.ros.org/wiki/xacro">
-  <!-- ros2_control System Hardware Interface Definition -->
-  <ros2_control name="DiffDriveSystem" type="system">
-    <hardware>
-      <!-- Option A: For Gazebo Sim (Harmonic) Simulation -->
-      <plugin>gz_ros2_control/GazeboSimSystem</plugin>
-      <!-- Option B: For Real Robot Hardware (Uncomment on real robot) -->
-      <!-- <plugin>my_robot_hardware/DiffDriveHardware</plugin> -->
-      <!-- <param name="serial_port">/dev/ttyUSB0</param> -->
-      <!-- <param name="baud_rate">115200</param> -->
-    </hardware>
-    <!-- Left Wheel Actuator Interface -->
-    <joint name="left_wheel_joint">
+<!--
+  Advanced Module 01: complete robot description for ros2_control.
+  Same geometry as the Essential track robot (Essential_ROS/Week_07 diff_drive_robot.urdf):
+  wheel radius 0.08 m, wheel separation 0.24 m. Self-contained on purpose: the Week 07 URDF
+  carries the gz DiffDrive system plugin, which would fight gz_ros2_control for the wheel joints.
+  The <ros2_control> block selects the hardware:
+    xacro diff_drive_ros2_control.xacro use_mock_hardware:=true   (default)
+        -> mock_components/GenericSystem : headless, no simulator, no robot.
+           calculate_dynamics integrates position from the commanded velocity,
+           so /joint_states and the odometry of diff_drive_controller really move.
+    xacro diff_drive_ros2_control.xacro use_mock_hardware:=false
+        -> gz_ros2_control/GazeboSimSystem : Gazebo Sim (Harmonic) drives the joints;
+           the gz_ros2_control plugin starts its own controller_manager with
+           the YAML given in controllers_file.
+  A real robot would use its own SystemInterface plugin here, e.g.
+    <plugin>my_robot_hardware/DiffDriveHardware</plugin>
+    <param name="serial_port">/dev/ttyUSB0</param>
+-->
+<robot name="amr_ros2_control" xmlns:xacro="http://www.ros.org/wiki/xacro">
+  <xacro:arg name="use_mock_hardware" default="true"/>
+  <xacro:arg name="controllers_file" default="$(find amr_adv01)/config/diff_drive_controller.yaml"/>
+  <!-- Geometry (keep in sync with config/diff_drive_controller.yaml; checked by test_description.py) -->
+  <xacro:property name="wheel_radius" value="0.08"/>
+  <xacro:property name="wheel_width" value="0.04"/>
+  <xacro:property name="wheel_separation" value="0.24"/>
+  <xacro:property name="wheel_mass" value="0.5"/>
+  <xacro:property name="base_length" value="0.40"/>
+  <xacro:property name="base_width" value="0.20"/>
+  <xacro:property name="base_height" value="0.10"/>
+  <xacro:property name="base_mass" value="5.0"/>
+  <xacro:property name="caster_radius" value="0.03"/>
+  <!-- Motor limit: 10 rad/s * 0.08 m = 0.8 m/s wheel rim speed -->
+  <xacro:property name="wheel_max_velocity" value="10.0"/>
+  <material name="chassis_blue"><color rgba="0.1 0.5 0.9 1.0"/></material>
+  <material name="wheel_dark"><color rgba="0.15 0.15 0.15 1.0"/></material>
+  <material name="caster_grey"><color rgba="0.6 0.6 0.6 1.0"/></material>
+  <!-- ===================== Links & joints ===================== -->
+  <link name="base_footprint"/>
+  <joint name="base_footprint_joint" type="fixed">
+    <parent link="base_footprint"/>
+    <child link="base_link"/>
+    <origin xyz="0 0 ${wheel_radius}" rpy="0 0 0"/>
+  </joint>
+  <link name="base_link">
+    <visual>
+      <origin xyz="0 0 0.02" rpy="0 0 0"/>
+      <geometry><box size="${base_length} ${base_width} ${base_height}"/></geometry>
+      <material name="chassis_blue"/>
+    </visual>
+    <collision>
+      <origin xyz="0 0 0.02" rpy="0 0 0"/>
+      <geometry><box size="${base_length} ${base_width} ${base_height}"/></geometry>
+    </collision>
+    <inertial>
+      <origin xyz="0 0 0.02" rpy="0 0 0"/>
+      <mass value="${base_mass}"/>
+      <inertia ixx="${base_mass / 12.0 * (base_width**2 + base_height**2)}" ixy="0" ixz="0"
+               iyy="${base_mass / 12.0 * (base_length**2 + base_height**2)}" iyz="0"
+               izz="${base_mass / 12.0 * (base_length**2 + base_width**2)}"/>
+    </inertial>
+  </link>
+  <!-- side: 1 = left (+y), -1 = right (-y) -->
+  <xacro:macro name="drive_wheel" params="prefix side">
+    <link name="${prefix}_wheel_link">
+      <visual>
+        <origin xyz="0 0 0" rpy="${-pi / 2} 0 0"/>
+        <geometry><cylinder radius="${wheel_radius}" length="${wheel_width}"/></geometry>
+        <material name="wheel_dark"/>
+      </visual>
+      <collision>
+        <origin xyz="0 0 0" rpy="${-pi / 2} 0 0"/>
+        <geometry><cylinder radius="${wheel_radius}" length="${wheel_width}"/></geometry>
+      </collision>
+      <inertial>
+        <origin xyz="0 0 0" rpy="${-pi / 2} 0 0"/>
+        <mass value="${wheel_mass}"/>
+        <inertia ixx="${wheel_mass / 12.0 * (3 * wheel_radius**2 + wheel_width**2)}" ixy="0" ixz="0"
+                 iyy="${wheel_mass / 12.0 * (3 * wheel_radius**2 + wheel_width**2)}" iyz="0"
+                 izz="${wheel_mass / 2.0 * wheel_radius**2}"/>
+      </inertial>
+    </link>
+    <joint name="${prefix}_wheel_joint" type="continuous">
+      <parent link="base_link"/>
+      <child link="${prefix}_wheel_link"/>
+      <origin xyz="0 ${side * wheel_separation / 2} 0" rpy="0 0 0"/>
+      <axis xyz="0 1 0"/>
+      <limit effort="10.0" velocity="${wheel_max_velocity}"/>
+    </joint>
+    <gazebo reference="${prefix}_wheel_link">
+      <mu1>1.0</mu1>
+      <mu2>1.0</mu2>
+    </gazebo>
+  </xacro:macro>
+  <xacro:drive_wheel prefix="left" side="1"/>
+  <xacro:drive_wheel prefix="right" side="-1"/>
+  <xacro:macro name="caster" params="prefix x">
+    <link name="${prefix}_caster_link">
+      <visual>
+        <geometry><sphere radius="${caster_radius}"/></geometry>
+        <material name="caster_grey"/>
+      </visual>
+      <collision>
+        <geometry><sphere radius="${caster_radius}"/></geometry>
+      </collision>
+      <inertial>
+        <mass value="0.1"/>
+        <inertia ixx="${0.4 * 0.1 * caster_radius**2}" ixy="0" ixz="0"
+                 iyy="${0.4 * 0.1 * caster_radius**2}" iyz="0" izz="${0.4 * 0.1 * caster_radius**2}"/>
+      </inertial>
+    </link>
+    <joint name="${prefix}_caster_joint" type="fixed">
+      <parent link="base_link"/>
+      <child link="${prefix}_caster_link"/>
+      <origin xyz="${x} 0 ${caster_radius - wheel_radius}" rpy="0 0 0"/>
+    </joint>
+    <!-- frictionless ball caster in Gazebo -->
+    <gazebo reference="${prefix}_caster_link">
+      <mu1>0.0</mu1>
+      <mu2>0.0</mu2>
+    </gazebo>
+  </xacro:macro>
+  <xacro:caster prefix="front" x="0.15"/>
+  <xacro:caster prefix="rear" x="-0.15"/>
+  <!-- ===================== ros2_control ===================== -->
+  <xacro:macro name="wheel_interfaces" params="joint">
+    <joint name="${joint}">
       <command_interface name="velocity">
-        <param name="min">-10.0</param>
-        <param name="max">10.0</param>
+        <param name="min">${-wheel_max_velocity}</param>
+        <param name="max">${wheel_max_velocity}</param>
       </command_interface>
       <state_interface name="position"/>
       <state_interface name="velocity"/>
     </joint>
-    <!-- Right Wheel Actuator Interface -->
-    <joint name="right_wheel_joint">
-      <command_interface name="velocity">
-        <param name="min">-10.0</param>
-        <param name="max">10.0</param>
-      </command_interface>
-      <state_interface name="position"/>
-      <state_interface name="velocity"/>
-    </joint>
+  </xacro:macro>
+  <ros2_control name="DiffDriveSystem" type="system">
+    <hardware>
+      <xacro:if value="$(arg use_mock_hardware)">
+        <plugin>mock_components/GenericSystem</plugin>
+        <!-- integrate position from the commanded velocity (otherwise position stays 0) -->
+        <param name="calculate_dynamics">true</param>
+      </xacro:if>
+      <xacro:unless value="$(arg use_mock_hardware)">
+        <plugin>gz_ros2_control/GazeboSimSystem</plugin>
+      </xacro:unless>
+    </hardware>
+    <xacro:wheel_interfaces joint="left_wheel_joint"/>
+    <xacro:wheel_interfaces joint="right_wheel_joint"/>
   </ros2_control>
-  <!-- Gazebo Sim ros2_control plugin integration -->
-  <gazebo>
-    <plugin filename="gz_ros2_control-system" name="gz_ros2_control::GazeboSimROS2ControlPlugin">
-      <parameters>$(find my_robot_bringup)/config/diff_drive_controller.yaml</parameters>
-    </plugin>
-  </gazebo>
+  <!-- Gazebo Sim loads the ros2_control system (its own controller_manager) from this plugin -->
+  <xacro:unless value="$(arg use_mock_hardware)">
+    <gazebo>
+      <plugin filename="gz_ros2_control-system" name="gz_ros2_control::GazeboSimROS2ControlPlugin">
+        <parameters>$(arg controllers_file)</parameters>
+      </plugin>
+    </gazebo>
+  </xacro:unless>
 </robot>

File: Essential_ROS/Week_07_URDF_Robot_Modeling/urdf/diff_drive_robot.urdf (robot description, URDF)
Before this commit: robot diff_drive_robot, 9 links, 8 joints
Links:
- link left_wheel_link: geometry collision sphere radius=0.08; visual cylinder length=0.04 radius=0.08
- link right_wheel_link: geometry collision sphere radius=0.08; visual cylinder length=0.04 radius=0.08
